File: hardware/pcb/placa_madre_esp32s3_uno/placa_madre_esp32s3_uno.kicad_pcb (KiCad board)
At the start: 4 copper layers, 195 x 159 mm, 128 parts, among them U1 74HCT541D, U10 ADS1115IDGSR, U2 ADS1115IDGSR, U3 MAX6675ISA+, U4 MAX6675ISA+, U5 MAX6675ISA+, U6 MAX6675ISA+, U7 MCP4725A0T-E/CH, U8 OPA2171AIDR, U9 OPA2171AIDR

Commit message: feat: add hardware manufacturing files and Gerber package for ESP32-S3 motherboard rev4
Parts:
- moved J_ENV 60.0 mm to (32.0, 120.0)
- moved J_HEATERS 35.6 mm to (186.0, 32.0), turned to -90 degrees
- moved J_TC 35.6 mm to (9.50, 108.0), turned to 90 degrees
- moved MH1 18.0 mm to (4.50, 4.50)
- moved MH2 18.0 mm to (190.5, 4.50)
- moved MH3 18.0 mm to (4.50, 154.5)
- moved MH4 18.0 mm to (190.5, 154.5)
- moved J_AC_IN 10.2 mm to (186.0, 12.0), turned to -90 degrees
- moved J_METER_I 10.2 mm to (186.0, 137.0), turned to -90 degrees
- moved J_METER_V 10.2 mm to (186.0, 119.5), turned to -90 degrees
- moved J_CELL 5.08 mm to (186.0, 78.0), turned to -90 degrees
- moved J_PWR_12V 5.08 mm to (186.0, 98.0), turned to -90 degrees
Connections:
- J_AC_IN pad 1: AC_EARTH -> AC_LINE
- J_AC_IN pad 3: AC_LINE -> AC_EARTH
- J_CELL pad 1: CELL_CATHODE -> CELL_ANODE
- J_CELL pad 2: CELL_ANODE -> CELL_CATHODE
- J_HEATERS pad 1: AC_NEUTRAL -> AC_T1
- J_HEATERS pad 2: AC_T4 -> AC_NEUTRAL
- J_HEATERS pad 3: AC_NEUTRAL -> AC_T2
- J_HEATERS pad 4: AC_T3 -> AC_NEUTRAL
- J_HEATERS pad 5: AC_NEUTRAL -> AC_T3
- J_HEATERS pad 6: AC_T2 -> AC_NEUTRAL
- J_HEATERS pad 7: AC_NEUTRAL -> AC_T4
- J_HEATERS pad 8: AC_T1 -> AC_NEUTRAL
- J_METER_I pad 1: ITOT_OUT -> +12V_VCSS
- J_METER_I pad 3: +12V_VCSS -> ITOT_OUT
- J_METER_V pad 1: VCELL_OUT -> +12V_VCSS
- J_METER_V pad 3: +12V_VCSS -> VCELL_OUT
- J_PWR_12V pad 1: PGND -> +12V_VCSS
- J_PWR_12V pad 2: +12V_VCSS -> PGND
- J_TC pad 1: TC0_POS -> AGND
- J_TC pad 2: AGND -> TC3_POS
- J_TC pad 3: TC1_POS -> AGND
- J_TC pad 4: AGND -> TC2_POS
- J_TC pad 5: TC2_POS -> AGND
- J_TC pad 6: AGND -> TC1_POS
- J_TC pad 7: TC3_POS -> AGND
- J_TC pad 8: AGND -> TC0_POS
Routing:
- net DGND: track 241.3 -> 300.5 mm, vias 4 -> 6
- net SHUNT2_SENSE: track 97.8 -> 95.3 mm
- net SHUNT1_SENSE: track 101.3 -> 99.3 mm
- net I2C_SCL: track 134.0 -> 132.9 mm
- net AGND: track 359.4 -> 358.4 mm
- net I2C_SDA: track 132.7 -> 131.8 mm, vias 6 -> 4
Other:
- board text removed: "+12V"
- board text removed: "+12V (Vcc)"
- board text removed: "+12V DC"
- board text removed: "+3V3"
- board text removed: "+5V"
- board text removed: "+ANODO"
- board text removed: "+ANODO (12V)"
- board text removed: "-CATODO"
- board text removed: "-CATODO (VCSS)"
- board text removed: "3V3 GND SCL SDA"
- board text removed: "AMPERIMETRO PANEL"
- board text removed: "CALEFACTORES 4 TINAS (AC)"
- board text removed: "CELDA HULL 267mL"
- board text removed: "COPROCESADOR AC ARDUINO NANO V3"
- board text removed: "FUENTE DC 12V 10A"
- board text removed: "GND"
- board text removed: "GND (0V)"
- board text removed: "H1"
- board text removed: "H2"
- board text removed: "H3"
- board text removed: "H3(HULL)"
- board text removed: "H4"
- board text removed: "I2C AMBIENTE (AHT20/BMP280)"
- board text removed: "I_OUT"
- board text removed: "I_SENSE (1 V/A)"
- board text removed: "L"
- board text removed: "L (Fase)"
- board text removed: "MODULO pH E201C"
- board text removed: "N"
- board text removed: "N (Neutro)"
- board text removed: "NODO MAESTRO ESP32-S3 (RTOS 2.0)"
- board text removed: "PE"
- board text removed: "PE (Tierra)"
- board text removed: "PLACA MADRE INDUSTRIAL PCBA REV 5.0 (ESP32-S3 + NANO)"
- board text removed: "PLANTA PILOTO DE ELECTRODEPOSICION Y GALVANOPLASTIA"
- board text removed: "RED AC 120/220V"
- board text removed: "STATUS RTOS"
- board text removed: "SUMIDERO VCSS BIPOLAR (2x IRLZ44N + RELE ZCS)"
- board text removed: "T1_L"
- board text removed: "T1_L (Desengrase)"
- board text removed: "T1_N"
- board text removed: "T1_N (Neutro)"
- board text removed: "T2_L"
- board text removed: "T2_L (Decapado)"
- board text removed: "T2_N"
- board text removed: "T2_N (Neutro)"
- board text removed: "T3_L (Celda Hull)"
- board text removed: "T3_L(HULL)"
- board text removed: "T3_N"
- board text removed: "T3_N (Neutro)"
- board text removed: "T4_L"
- board text removed: "T4_L (Niquelado)"
- board text removed: "T4_N"
- board text removed: "T4_N (Neutro)"
- board text removed: "TC1 + (Desengrase)"
- board text removed: "TC1 - (AGND)"
- board text removed: "TC1+"
- board text removed: "TC1-"
- board text removed: "TC2 + (Decapado)"
- board text removed: "TC2 - (AGND)"
- board text removed: "TC2+"
- board text removed: "TC2-"
- board text removed: "TC3 + (Celda Hull)"
- board text removed: "TC3 - (AGND)"
- board text removed: "TC3+(HULL)"
- board text removed: "TC3-"
- board text removed: "TC4 + (Niquelado)"
- board text removed: "TC4 - (AGND)"
- board text removed: "TC4+"
- board text removed: "TC4-"
- board text removed: "TERMOPARES K (MAX6675)"
- board text removed: "VCC GND Po Do To GND"
- board text removed: "VCSS"
- board text removed: "VCSS_ON"
- board text removed: "VOLTIMETRO PANEL"
- board text removed: "V_OUT"
- board text removed: "V_SENSE (0-30V)"
- board text removed: "ZONA AC 120V - 4x TRIACs BTA24"
- board text removed: "ZONA AC 120V/220V - 4x TRIACs BTA24"
- board text removed: "[AMPERIMETRO PANEL]"
- board text removed: "[CALEFACTORES 4 TINAS]"
- board text removed: "[CELDA HULL 267mL]"
- board text removed: "[FUENTE DC 12V 10A]"
- board text removed: "[I2C AMBIENTE]"
- board text removed: "[RED AC 120/220V]"
- board text removed: "[SONDA pH E201C]"
- board text removed: "[TERMOPARES K (MAX6675)]"
- board text removed: "[VOLTIMETRO PANEL]"
